Commit message: ADD: revert the process last night

File: install/humanoid_v1/share/humanoid_v1/urdf/robot.urdf.xacro (robot description, xacro)
@@ -3,262 +3,229 @@
 <joint name="base_link_to_base" type="fixed">
 <parent link="base_link"/>
-<child link="hip_x_mount" />
+<child link="base" />
 <origin rpy="0.0 0 0" xyz="0 0 0"/>
 </joint>
-<link name="hip_x_mount">
-<visual>
-<origin xyz="0 0 0" rpy="0 -0 0" />
-<geometry>
-<mesh filename="package://humanoid_v1/meshes/part_2.stl"/>
-</geometry>
-<material name="part_2_material">
-<color rgba="0 0 0 1.0"/>
-</material>
-</visual>
-<collision>
-<origin xyz="0 0 0" rpy="0 -0 0" />
-<geometry>
-<mesh filename="package://humanoid_v1/meshes/part_2.stl"/>
-</geometry>
-<material name="part_2_material">
-<color rgba="0 0 0 1.0"/>
-</material>
-</collision>
-<visual>
-<origin xyz="0 0 0" rpy="0 -0 0" />
-<geometry>
-<mesh filename="package://humanoid_v1/meshes/part_1.stl"/>
-</geometry>
-<material name="part_1_material">
-<color rgba="0 0 0 1.0"/>
-</material>
-</visual>
-<collision>
-<origin xyz="0 0 0" rpy="0 -0 0" />
-<geometry>
-<mesh filename="package://humanoid_v1/meshes/part_1.stl"/>
-</geometry>
-<material name="part_1_material">
-<color rgba="0 0 0 1.0"/>
-</material>
-</collision>
-<visual>
-<origin xyz="0.065 1.30104e-18 -0.056" rpy="-6.0021e-16 -1.83761e-31 -1.5708" />
-<geometry>
-<mesh filename="package://humanoid_v1/meshes/housing.stl"/>
-</geometry>
-<material name="housing_material">
-<color rgba="0.964706 0.964706 0.952941 1.0"/>
-</material>
-</visual>
-<collision>
-<origin xyz="0.065 1.30104e-18 -0.056" rpy="-6.0021e-16 -1.83761e-31 -1.5708" />
-<geometry>
-<mesh filename="package://humanoid_v1/meshes/housing.stl"/>
-</geometry>
-<material name="housing_material">
-<color rgba="0.964706 0.964706 0.952941 1.0"/>
-</material>
-</collision>
-<visual>
-<origin xyz="0 0 0" rpy="0 -0 0" />
-<geometry>
-<mesh filename="package://humanoid_v1/meshes/part_4.stl"/>
-</geometry>
-<material name="part_4_material">
-<color rgba="0 0 0 1.0"/>
-</material>
-</visual>
-<collision>
-<origin xyz="0 0 0" rpy="0 -0 0" />
-<geometry>
-<mesh filename="package://humanoid_v1/meshes/part_4.stl"/>
-</geometry>
-<material name="part_4_material">
-<color rgba="0 0 0 1.0"/>
-</material>
-</collision>
-<visual>
-<origin xyz="0 0 0" rpy="0 -0 0" />
-<geometry>
-<mesh filename="package://humanoid_v1/meshes/x.stl"/>
-</geometry>
-<material name="x_material">
-<color rgba="1 0 0 1.0"/>
-</material>
-</visual>
-<collision>
-<origin xyz="0 0 0" rpy="0 -0 0" />
-<geometry>
-<mesh filename="package://humanoid_v1/meshes/x.stl"/>
-</geometry>
-<material name="x_material">
-<color rgba="1 0 0 1.0"/>
-</material>
-</collision>
-<visual>
-<origin xyz="0 0 0" rpy="0 -0 0" />
-<geometry>
-<mesh filename="package://humanoid_v1/meshes/z.stl"/>
-</geometry>
-<material name="z_material">
-<color rgba="0.231373 0.380392 0.705882 1.0"/>
-</material>
-</visual>
-<collision>
-<origin xyz="0 0 0" rpy="0 -0 0" />
-<geometry>
-<mesh filename="package://humanoid_v1/meshes/z.stl"/>
-</geometry>
-<material name="z_material">
-<color rgba="0.231373 0.380392 0.705882 1.0"/>
-</material>
-</collision>
-<visual>
-<origin xyz="0 0 0" rpy="0 -0 0" />
-<geometry>
-<mesh filename="package://humanoid_v1/meshes/part_3.stl"/>
-</geometry>
-<material name="part_3_material">
-<color rgba="0 0 0 1.0"/>
-</material>
-</visual>
-<collision>
-<origin xyz="0 0 0" rpy="0 -0 0" />
-<geometry>
-<mesh filename="package://humanoid_v1/meshes/part_3.stl"/>
-</geometry>
-<material name="part_3_material">
-<color rgba="0 0 0 1.0"/>
-</material>
-</collision>
-<visual>
-<origin xyz="0 0 0" rpy="0 -0 0" />
-<geometry>
-<mesh filename="package://humanoid_v1/meshes/part_4.stl"/>
-</geometry>
-<material name="part_4_material">
-<color rgba="0.917647 0.917647 0.917647 1.0"/>
-</material>
-</visual>
-<collision>
-<origin xyz="0 0 0" rpy="0 -0 0" />
-<geometry>
-<mesh filename="package://humanoid_v1/meshes/part_4.stl"/>
-</geometry>
-<material name="part_4_material">
-<color rgba="0.917647 0.917647 0.917647 1.0"/>
-</material>
-</collision>
-<visual>
-<origin xyz="0 0 0" rpy="0 -0 0" />
-<geometry>
-<mesh filename="package://humanoid_v1/meshes/part_5.stl"/>
-</geometry>
-<material name="part_5_material">
-<color rgba="0.917647 0.917647 0.917647 1.0"/>
-</material>
-</visual>
-<collision>
-<origin xyz="0 0 0" rpy="0 -0 0" />
-<geometry>
-<mesh filename="package://humanoid_v1/meshes/part_5.stl"/>
-</geometry>
-<material name="part_5_material">
-<color rgba="0.917647 0.917647 0.917647 1.0"/>
-</material>
-</collision>
-<visual>
-<origin xyz="0 0 0" rpy="0 -0 0" />
-<geometry>
-<mesh filename="package://humanoid_v1/meshes/y.stl"/>
-</geometry>
-<material name="y_material">
-<color rgba="0.372549 0.654902 0.239216 1.0"/>
-</material>
-</visual>
-<collision>
-<origin xyz="0 0 0" rpy="0 -0 0" />
-<geometry>
-<mesh filename="package://humanoid_v1/meshes/y.stl"/>
-</geometry>
-<material name="y_material">
-<color rgba="0.372549 0.654902 0.239216 1.0"/>
-</material>
-</collision>
-<visual>
-<origin xyz="0 0 0" rpy="0 -0 0" />
-<geometry>
-<mesh filename="package://humanoid_v1/meshes/part_6.stl"/>
-</geometry>
-<material name="part_6_material">
-<color rgba="0.917647 0.917647 0.917647 1.0"/>
-</material>
-</visual>
-<collision>
-<origin xyz="0 0 0" rpy="0 -0 0" />
-<geometry>
-<mesh filename="package://humanoid_v1/meshes/part_6.stl"/>
-</geometry>
-<material name="part_6_material">
-<color rgba="0.917647 0.917647 0.917647 1.0"/>
-</material>
-</collision>
-<visual>
-<origin xyz="0.065 1.30104e-18 -0.056" rpy="-6.0021e-16 -1.83761e-31 -1.5708" />
-<geometry>
-<mesh filename="package://humanoid_v1/meshes/housing.stl"/>
-</geometry>
-<material name="housing_material">
-<color rgba="0.964706 0.964706 0.952941 1.0"/>
-</material>
-</visual>
-<collision>
-<origin xyz="0.065 1.30104e-18 -0.056" rpy="-6.0021e-16 -1.83761e-31 -1.5708" />
-<geometry>
-<mesh filename="package://humanoid_v1/meshes/housing.stl"/>
-</geometry>
-<material name="housing_material">
-<color rgba="0.964706 0.964706 0.952941 1.0"/>
-</material>
-</collision>
-<inertial>
-<origin xyz="0.0218905 -7.94313e-13 -0.012103" rpy="0 0 0"/>
-<mass value="0.325819" />
-<inertia ixx="0.000847428" ixy="1.47161e-14"  ixz="0.000181898" iyy="0.00117214" iyz="-1.18597e-14" izz="0.00157896" />
-</inertial>
-</link>
-<link name="hip_y_mount">
-<visual>
-<origin xyz="0 0 0" rpy="-1.5708 -0 8.97521e-48" />
-<geometry>
-<mesh filename="package://humanoid_v1/meshes/component1.stl"/>
-</geometry>
-<material name="component1_material">
-<color rgba="0.964706 0.964706 0.952941 1.0"/>
-</material>
-</visual>
-<collision>
-<origin xyz="0 0 0" rpy="-1.5708 -0 8.97521e-48" />
-<geometry>
-<mesh filename="package://humanoid_v1/meshes/component1.stl"/>
-</geometry>
-<material name="component1_material">
-<color rgba="0.964706 0.964706 0.952941 1.0"/>
-</material>
-</collision>
-<inertial>
-<origin xyz="-1.12795e-08 3.38727e-09 -0.0357636" rpy="0 0 0"/>
-<mass value="0.0763972" />
-<inertia ixx="0.000122996" ixy="-1.23623e-11"  ixz="1.3626e-11" iyy="8.31952e-05" iyz="-6.33605e-12" izz="5.09352e-05" />
-</inertial>
-</link>
-<joint name="upperleg_x_r_joint" type="revolute">
-<origin xyz="0.08 -3.46945e-18 -0.056" rpy="-1.5708 1.83761e-31 1.5708" />
-<parent link="hip_x_mount" />
-<child link="hip_y_mount" />
+<link name="base">
+<visual>
+<origin xyz="0 0 0" rpy="0 -0 0" />
+<geometry>
+<mesh filename="package://humanoid_v1/meshes/base_visual.stl"/>
+</geometry>
+<material name="base_material">
+<color rgba="0.8 0.8 0.8 1.0"/>
+</material>
+</visual>
+<collision>
+<origin xyz="0 0 0" rpy="0 -0 0" />
+<geometry>
+<mesh filename="package://humanoid_v1/meshes/base_collision.stl"/>
+</geometry>
+<material name="base_material">
+<color rgba="0.5 0.5 0.5 1.0"/>
+</material>
+</collision>
+<inertial>
+<origin xyz="7.3655e-18 -0.010053 -0.00364106" rpy="0 0 0"/>
+<mass value="2.09484" />
+<inertia ixx="0.0277752" ixy="4.21566e-12"  ixz="2.80707e-18" iyy="0.0322146" iyz="0.00449915" izz="0.00921242" />
+</inertial>
+</link>
+<link name="upperlegx">
+<visual>
+<origin xyz="0 0 0" rpy="0 -0 0" />
+<geometry>
+<mesh filename="package://humanoid_v1/meshes/upperlegx_visual.stl"/>
+</geometry>
+<material name="upperlegx_material">
+<color rgba="0.8 0.8 0.8 1.0"/>
+</material>
+</visual>
+<collision>
+<origin xyz="0 0 0" rpy="0 -0 0" />
+<geometry>
+<mesh filename="package://humanoid_v1/meshes/upperlegx_collision.stl"/>
+</geometry>
+<material name="upperlegx_material">
+<color rgba="0.5 0.5 0.5 1.0"/>
+</material>
+</collision>
+<inertial>
+<origin xyz="0.0134137 -2.72625e-09 -0.0503059" rpy="0 0 0"/>
+<mass value="0.732188" />
+<inertia ixx="0.000759087" ixy="1.06686e-07"  ixz="1.66386e-05" iyy="0.000618258" iyz="-1.55325e-11" izz="0.000568045" />
+</inertial>
+</link>
+<link name="upperlegy">
+<visual>
+<origin xyz="0 0 0" rpy="0 -0 0" />
+<geometry>
+<mesh filename="package://humanoid_v1/meshes/upperlegy_visual.stl"/>
+</geometry>
+<material name="upperlegy_material">
+<color rgba="0.8 0.8 0.8 1.0"/>
+</material>
+</visual>
+<collision>
+<origin xyz="0 0 0" rpy="0 -0 0" />
+<geometry>
+<mesh filename="package://humanoid_v1/meshes/upperlegy_collision.stl"/>
+</geometry>
+<material name="upperlegy_material">
+<color rgba="0.5 0.5 0.5 1.0"/>
+</material>
+</collision>
+<inertial>
+<origin xyz="-3.43844e-09 0.109524 -0.0175" rpy="0 0 0"/>
+<mass value="0.65579" />
+<inertia ixx="0.000501677" ixy="-1.06691e-07"  ixz="-1.61313e-12" iyy="0.000618053" iyz="2.08745e-12" izz="0.000501763" />
+</inertial>
+</link>
+<link name="upperlegz">
+<visual>
+<origin xyz="0 0 0" rpy="0 -0 0" />
+<geometry>
+<mesh filename="package://humanoid_v1/meshes/upperlegz_visual.stl"/>
+</geometry>
+<material name="upperlegz_material">
+<color rgba="0.8 0.8 0.8 1.0"/>
+</material>
+</visual>
+<collision>
+<origin xyz="0 0 0" rpy="0 -0 0" />
+<geometry>
+<mesh filename="package://humanoid_v1/meshes/upperlegz_collision.stl"/>
+</geometry>
+<material name="upperlegz_material">
+<color rgba="0.5 0.5 0.5 1.0"/>
+</material>
+</collision>
+<inertial>
+<origin xyz="0.00580914 -0.000686366 0.226874" rpy="0 0 0"/>
+<mass value="1.07815" />
+<inertia ixx="0.0108106" ixy="1.34037e-05"  ixz="-0.000206513" iyy="0.0107895" iyz="5.82774e-07" izz="0.000764981" />
+</inertial>
+</link>
+<joint name="upperleg_z_r" type="revolute">
+<origin xyz="-5.27356e-16 0.142 -0.0175" rpy="-1.5708 -1.65983e-14 7.69755e-15" />
+<parent link="upperlegy" />
+<child link="upperlegz" />
 <axis xyz="0 0 1"/>
 <limit effort="1" velocity="20" lower="-1.5708" upper="1.5708"/>
 <joint_properties friction="0.0"/>
 </joint>
+<joint name="upperleg_y_r" type="revolute">
+<origin xyz="-0.0175 -4.54498e-15 -0.052" rpy="-3.14159 1.5708 0" />
+<parent link="upperlegx" />
+<child link="upperlegy" />
+<axis xyz="0 0 1"/>
+<limit effort="1" velocity="20" lower="-6.28319" upper="6.28319"/>
+<joint_properties friction="0.0"/>
+</joint>
+<joint name="upperleg_x_r" type="revolute">
+<origin xyz="0.083 2.90452e-17 -0.056" rpy="1.5708 -3.55271e-15 -1.5708" />
+<parent link="base" />
+<child link="upperlegx" />
+<axis xyz="0 0 1"/>
+<limit effort="1" velocity="20" lower="-6.28319" upper="6.28319"/>
+<joint_properties friction="0.0"/>
+</joint>
+<link name="upperlegx_2">
+<visual>
+<origin xyz="0 0 0" rpy="0 -0 0" />
+<geometry>
+<mesh filename="package://humanoid_v1/meshes/upperlegx_2_visual.stl"/>
+</geometry>
+<material name="upperlegx_2_material">
+<color rgba="0.8 0.8 0.8 1.0"/>
+</material>
+</visual>
+<collision>
+<origin xyz="0 0 0" rpy="0 -0 0" />
+<geometry>
+<mesh filename="package://humanoid_v1/meshes/upperlegx_2_collision.stl"/>
+</geometry>
+<material name="upperlegx_2_material">
+<color rgba="0.5 0.5 0.5 1.0"/>
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
File: onshape/humanoid_v1/robot.urdf (robot description, URDF)
Before this commit: robot humanoid_v1, 3 links, 2 joints
Links:
- removed link hip_x_mount
- removed link hip_y_mount
- added link base, mass 2.09484; collision mesh filename=package:///base_collision.stl; visual mesh filename=package:///base_visual.stl
- added link upperlegx, mass 0.732188; collision mesh filename=package:///upperlegx_collision.stl; visual mesh filename=package:///upperlegx_visual.stl
- added link upperlegx_2, mass 0.732188; collision mesh filename=package:///upperlegx_2_collision.stl; visual mesh filename=package:///upperlegx_2_visual.stl
- added link upperlegy, mass 0.65579; collision mesh filename=package:///upperlegy_collision.stl; visual mesh filename=package:///upperlegy_visual.stl
- added link upperlegy_2, mass 0.65579; collision mesh filename=package:///upperlegy_2_collision.stl; visual mesh filename=package:///upperlegy_2_visual.stl
- added link upperlegz, mass 1.07815; collision mesh filename=package:///upperlegz_collision.stl; visual mesh filename=package:///upperlegz_visual.stl
- added link upperlegz_copy_1, mass 1.07815; collision mesh filename=package:///upperlegz_copy_1_collision.stl; visual mesh filename=package:///upperlegz_copy_1_visual.stl
Joints:
- removed joint upperleg_x_r_joint
- added joint upperleg_x_l: type revolute, parent base, child upperlegx_2, origin xyz=-0.083 -1.69021e-17 -0.056 rpy=-1.5708 -3.77261e-29 -1.5708, axis 0 0 1, limit lower=-6.28319 upper=6.28319 effort=1 velocity=20
- added joint upperleg_x_r: type revolute, parent base, child upperlegx, origin xyz=0.083 2.90452e-17 -0.056 rpy=1.5708 -3.55271e-15 -1.5708, axis 0 0 1, limit lower=-6.28319 upper=6.28319 effort=1 velocity=20
- added joint upperleg_y_l: type revolute, parent upperlegx_2, child upperlegy_2, origin xyz=-0.0175 -4.16334e-17 -0.052 rpy=6.12323e-17 -1.5708 0, axis 0 0 1, limit lower=-6.28319 upper=6.28319 effort=1 velocity=20
- added joint upperleg_y_r: type revolute, parent upperlegx, child upperlegy, origin xyz=-0.0175 -4.54498e-15 -0.052 rpy=-3.14159 1.5708 0, axis 0 0 1, limit lower=-6.28319 upper=6.28319 effort=1 velocity=20
- added joint upperleg_z_l: type revolute, parent upperlegy_2, child upperlegz_copy_1, origin xyz=-4.71845e-16 0.142 -0.0175 rpy=-1.5708 -2.15921e-15 7.69755e-15, axis 0 0 1, limit lower=-1.5708 upper=1.5708 effort=1 velocity=20
- added joint upperleg_z_r: type revolute, parent upperlegy, child upperlegz, origin xyz=-5.27356e-16 0.142 -0.0175 rpy=-1.5708 -1.65983e-14 7.69755e-15, axis 0 0 1, limit lower=-1.5708 upper=1.5708 effort=1 velocity=20
- joint base_link_to_base: child hip_x_mount -> base
