Commit message: ADD: almost finish leg

File: install/humanoid_v1/share/humanoid_v1/urdf/robot.urdf.xacro (robot description, xacro)
@@ -7,4 +7,194 @@
 </joint>
 <link name="base">
+<!-- Shapes for extrusion_150mm -->
+<collision>
+<origin xyz="0 0.06 0" rpy="0 -0 0" />
+<geometry>
+<box size="0.15 0.02 0.02" />
+</geometry>
+</collision>
+<collision>
+<origin xyz="0 -0.06 0" rpy="0 -0 0" />
+<geometry>
+<box size="0.15 0.02 0.02" />
+</geometry>
+</collision>
+<!-- Shapes for housing -->
+<collision>
+<origin xyz="-0.05 6.73073e-18 -0.056" rpy="1.5708 -0 1.5708" />
+<geometry>
+<cylinder length="0.02" radius="0.045" />
+</geometry>
+</collision>
+<!-- Shapes for part_2 -->
+<collision>
+<origin xyz="0.04 1.88738e-17 -0.056" rpy="-3.14159 -1.5708 0" />
+<geometry>
+<cylinder length="0.022" radius="0.036" />
+</geometry>
+</collision>
+<!-- Shapes for part_2 -->
+<collision>
+<origin xyz="-0.04 -1.56752e-17 -0.056" rpy="4.17605e-18 -1.5708 0" />
+<geometry>
+<cylinder length="0.022" radius="0.036" />
+</geometry>
+</collision>
+<!-- Shapes for part_1 -->
+<collision>
+<origin xyz="0.034 0 -0.056" rpy="-3.14159 -1.5708 0" />
+<geometry>
+<cylinder length="0.018" radius="0.024" />
+</geometry>
+</collision>
+<!-- Shapes for housing -->
+<collision>
+<origin xyz="-0.066 6.93889e-18 -0.056" rpy="-3.14159 -1.5708 0" />
+<geometry>
+<cylinder length="0.02" radius="0.045" />
+</geometry>
+</collision>
+<!-- Shapes for extrusion_400mm -->
+<collision>
+<origin xyz="0.065 -0.06 0.21" rpy="0 -0 0" />
+<geometry>
+<box size="0.02 0.02 0.4" />
+</geometry>
+</collision>
+<collision>
+<origin xyz="-0.065 -0.06 0.21" rpy="0 -0 0" />
+<geometry>
+<box size="0.02 0.02 0.4" />
+</geometry>
+</collision>
+<!-- Shapes for housing -->
+<collision>
+<origin xyz="0.05 -6.73073e-18 -0.056" rpy="1.5708 -0 -1.5708" />
+<geometry>
+<cylinder length="0.02" radius="0.045" />
+</geometry>
+</collision>
+<!-- Shapes for extrusion_400mm -->
+<collision>
+<origin xyz="0.065 -0.06 0.21" rpy="0 -0 0" />
+<geometry>
+<box size="0.02 0.02 0.4" />
+</geometry>
+</collision>
+<collision>
+<origin xyz="-0.065 -0.06 0.21" rpy="0 -0 0" />
+<geometry>
+<box size="0.02 0.02 0.4" />
+</geometry>
+</collision>
+<!-- Shapes for motor_shell -->
+<collision>
+<origin xyz="0.035 0 -0.056" rpy="-0 -1.5708 0" />
+<geometry>
+<cylinder length="0.03" radius="0.045" />
+</geometry>
+</collision>
+<!-- Shapes for housing -->
+<collision>
+<origin xyz="0.066 0 -0.056" rpy="-0 -1.5708 0" />
+<geometry>
+<cylinder length="0.02" radius="0.045" />
+</geometry>
+</collision>
+<!-- Shapes for motor_shell -->
+<collision>
+<origin xyz="-0.035 6.93889e-18 -0.056" rpy="-3.14159 -1.5708 0" />
+<geometry>
+<cylinder length="0.03" radius="0.045" />
+</geometry>
+</collision>
+<!-- Shapes for extrusion_100mm -->
+<collision>
+<origin xyz="0.065 0 0" rpy="0 -0 0" />
+<geometry>
+<box size="0.02 0.1 0.02" />
+</geometry>
+</collision>
+<collision>
+<origin xyz="-0.065 0 0" rpy="0 -0 0" />
+<geometry>
+<box size="0.02 0.1 0.02" />
+</geometry>
+</collision>
+<!-- Shapes for housing -->
+<collision>
+<origin xyz="-0.066 6.93889e-18 -0.056" rpy="-3.14159 -1.5708 0" />
+<geometry>
+<cylinder length="0.02" radius="0.045" />
+</geometry>
+</collision>
+<!-- Shapes for housing -->
+<collision>
+<origin xyz="0.066 0 -0.056" rpy="-0 -1.5708 0" />
+<geometry>
+<cylinder length="0.02" radius="0.045" />
+</geometry>
+</collision>
+<!-- Shapes for part_1 -->
+<collision>
+<origin xyz="-0.034 0 -0.056" rpy="-0 -1.5708 0" />
+<geometry>
+<cylinder length="0.018" radius="0.024" />
+</geometry>
+</collision>
+<!-- Shapes for housing -->
+<collision>
+<origin xyz="-0.05 6.73073e-18 -0.056" rpy="1.5708 -0 1.5708" />
+<geometry>
+<cylinder length="0.02" radius="0.045" />
+</geometry>
+</collision>
+<!-- Shapes for extrusion_150mm -->
+<collision>
+<origin xyz="0 0.06 0" rpy="0 -0 0" />
+<geometry>
+<box size="0.15 0.02 0.02" />
+</geometry>
+</collision>
+<collision>
+<origin xyz="0 -0.06 0" rpy="0 -0 0" />
+<geometry>
+<box size="0.15 0.02 0.02" />
+</geometry>
+</collision>
+<!-- Shapes for housing -->
+<collision>
+<origin xyz="0.05 -6.73073e-18 -0.056" rpy="1.5708 -0 -1.5708" />
+<geometry>
+<cylinder length="0.02" radius="0.045" />
+</geometry>
+</collision>
+<!-- Shapes for extrusion_100mm -->
+<collision>
+<origin xyz="0.065 0 0" rpy="0 -0 0" />
+<geometry>
+<box size="0.02 0.1 0.02" />
+</geometry>
+</collision>
+<collision>
+<origin xyz="-0.065 0 0" rpy="0 -0 0" />
+<geometry>
+<box size="0.02 0.1 0.02" />
+</geometry>
+</collision>
+<!-- Shapes for housing -->
+<collision>
+<origin xyz="0.066 0 -0.056" rpy="-0 -1.5708 0" />
+<geometry>
+<cylinder length="0.02" radius="0.045" />
+</geometry>
+</collision>
+<!-- Shapes for housing -->
+<collision>
+<origin xyz="-0.066 6.93889e-18 -0.056" rpy="-3.14159 -1.5708 0" />
+<geometry>
+<cylinder length="0.02" radius="0.045" />
+</geometry>
+</collision>
 <visual>
 <origin xyz="0 0 0" rpy="0 -0 0" />
@@ -26,10 +216,52 @@
 </collision>
 <inertial>
-<origin xyz="7.3655e-18 -0.010053 -0.00364106" rpy="0 0 0"/>
+<origin xyz="7.77955e-18 -0.010053 -0.00364106" rpy="0 0 0"/>
 <mass value="2.09484" />
-<inertia ixx="0.0277752" ixy="4.21566e-12"  ixz="2.80707e-18" iyy="0.0322146" iyz="0.00449915" izz="0.00921242" />
+<inertia ixx="0.0277752" ixy="4.21566e-12"  ixz="2.12902e-18" iyy="0.0322146" iyz="0.00449915" izz="0.00921242" />
 </inertial>
 </link>
 <link name="upperlegx">
+<!-- Shapes for motor_shell -->
+<collision>
+<origin xyz="0.0305 -5.23454e-15 -0.052" rpy="1.5708 1.22125e-15 1.5708" />
+<geometry>
+<cylinder length="0.03" radius="0.045" />
+</geometry>
+</collision>
+<!-- Shapes for part_1 -->
+<collision>
+<origin xyz="0.0315 -4.9426e-15 -0.052" rpy="-1.5708 1.80744e-13 1.5708" />
+<geometry>
+<cylinder length="0.018" radius="0.024" />
+</geometry>
+</collision>
+<!-- Shapes for housing -->
+<collision>
+<origin xyz="-0.0005 -4.8353e-15 -0.052" rpy="1.5708 1.22125e-15 1.5708" />
+<geometry>
+<cylinder length="0.02" radius="0.045" />
+</geometry>
+</collision>
+<!-- Shapes for part_2 -->
+<collision>
+<origin xyz="0.0255 -4.87277e-15 -0.052" rpy="-1.5708 1.57763e-13 1.5708" />
+<geometry>
+<cylinder length="0.022" radius="0.036" />
+</geometry>
+</collision>
+<!-- Shapes for housing -->
+<collision>
+<origin xyz="-0.0005 -4.8353e-15 -0.052" rpy="1.5708 1.22125e-15 1.5708" />
+<geometry>
+<cylinder length="0.02" radius="0.045" />
+</geometry>
+</collision>
+<!-- Shapes for housing -->
+<collision>
+<origin xyz="-0.0005 -4.8353e-15 -0.052" rpy="1.5708 1.22125e-15 1.5708" />
+<geometry>
+<cylinder length="0.02" radius="0.045" />
+</geometry>
+</collision>
 <visual>
 <origin xyz="0 0 0" rpy="0 -0 0" />
@@ -57,4 +289,46 @@
 </link>
 <link name="upperlegy">
+<!-- Shapes for part_2 -->
+<collision>
+<origin xyz="-1.74434e-16 0.099 -0.0175" rpy="-1.5708 -1.68759e-14 7.69755e-15" />
+<geometry>
+<cylinder length="0.022" radius="0.036" />
+</geometry>
+</collision>
+<!-- Shapes for housing -->
+<collision>
+<origin xyz="-3.79141e-16 0.125 -0.0175" rpy="1.5708 3.15544e-30 7.69755e-15" />
+<geometry>
+<cylinder length="0.02" radius="0.045" />
+</geometry>
+</collision>
+<!-- Shapes for housing -->
+<collision>
+<origin xyz="-3.79141e-16 0.125 -0.0175" rpy="1.5708 3.15544e-30 7.69755e-15" />
+<geometry>
+<cylinder length="0.02" radius="0.045" />
+</geometry>
+</collision>
+<!-- Shapes for part_1 -->
+<collision>
+<origin xyz="-1.27787e-16 0.093 -0.0175" rpy="-1.5708 3.15544e-30 7.69755e-15" />
+<geometry>
+<cylinder length="0.018" radius="0.024" />
+</geometry>
+</collision>
+<!-- Shapes for motor_shell -->
+<collision>
+<origin xyz="-1.30192e-16 0.094 -0.0175" rpy="1.5708 3.15544e-30 7.69755e-15" />
+<geometry>
+<cylinder length="0.03" radius="0.045" />
+</geometry>
+</collision>
+<!-- Shapes for housing -->
+<collision>
+<origin xyz="-3.79141e-16 0.125 -0.0175" rpy="1.5708 3.15544e-30 7.69755e-15" />
+<geometry>
+<cylinder length="0.02" radius="0.045" />
+</geometry>
+</collision>
 <visual>
 <origin xyz="0 0 0" rpy="0 -0 0" />
@@ -82,4 +356,46 @@
 </link>
 <link name="upperlegz">
+<!-- Shapes for motor_shell -->
+<collision>
+<origin xyz="-0.011 1.22216e-18 0.288" rpy="-0 -1.5708 0" />
+<geometry>
+<cylinder length="0.03" radius="0.045" />
+</geometry>
+</collision>
+<!-- Shapes for housing -->
+<collision>
+<origin xyz="0.02 1.22216e-18 0.288" rpy="-0 -1.5708 0" />
+<geometry>
+<cylinder length="0.02" radius="0.045" />
+</geometry>
+</collision>
+<!-- Shapes for housing -->
+<collision>
+<origin xyz="0.02 1.22216e-18 0.288" rpy="-0 -1.5708 0" />
+<geometry>
+<cylinder length="0.02" radius="0.045" />
+</geometry>
+</collision>
+<!-- Shapes for part_1 -->
+<collision>
+<origin xyz="-0.012 1.22134e-17 0.288" rpy="-3.14159 -1.5708 0" />
+<geometry>
+<cylinder length="0.018" radius="0.024" />
+</geometry>
+</collision>
+<!-- Shapes for part_2 -->
+<collision>
+<origin xyz="-0.006 -1.60178e-18 0.288" rpy="-3.14159 -1.5708 0" />
+<geometry>
+<cylinder length="0.022" radius="0.036" />
+</geometry>
+</collision>
+<!-- Shapes for housing -->
+<collision>
+<origin xyz="0.02 1.22216e-18 0.288" rpy="-0 -1.5708 0" />
+<geometry>
+<cylinder length="0.02" radius="0.045" />
+</geometry>
+</collision>
 <visual>
 <origin xyz="0 0 0" rpy="0 -0 0" />
@@ -106,4 +422,154 @@
 </inertial>
 </link>
+<link name="lowerlegx">
+<!-- Shapes for housing -->
+<collision>
+<origin xyz="1.19838e-19 0.123 0.037" rpy="1.5708 1.5708 0" />
+<geometry>
+<cylinder length="0.02" radius="0.045" />
+</geometry>
+</collision>
+<!-- Shapes for housing -->
+<collision>
+<origin xyz="1.19838e-19 0.123 0.037" rpy="1.5708 1.5708 0" />
+<geometry>
+<cylinder length="0.02" radius="0.045" />
+</geometry>
+</collision>
+<!-- Shapes for housing -->
+<collision>
+<origin xyz="1.19838e-19 0.123 0.037" rpy="1.5708 1.5708 0" />
+<geometry>
+<cylinder length="0.02" radius="0.045" />
+</geometry>
+</collision>
+<!-- Shapes for part_2 -->
+<collision>
+<origin xyz="-1.15666e-17 0.1 0.037" rpy="-1.5708 1.5708 0" />
+<geometry>
+<cylinder length="0.022" radius="0.036" />
+</geometry>
+</collision>
+<!-- Shapes for part_1 -->
+<collision>
+<origin xyz="-1.17871e-17 0.093 0.037" rpy="-1.5708 1.5708 0" />
+<geometry>
+<cylinder length="0.018" radius="0.024" />
+</geometry>
+</collision>
+<!-- Shapes for motor_shell -->
+<collision>
+<origin xyz="1.19838e-19 0.092 0.037" rpy="1.5708 1.5708 0" />
+<geometry>
+<cylinder length="0.03" radius="0.045" />
+</geometry>
+</collision>
+<visual>
+<origin xyz="0 0 0" rpy="0 -0 0" />
+<geometry>
+<mesh filename="package://humanoid_v1/meshes/lowerlegx_visual.stl"/>
+</geometry>
+<material name="lowerlegx_material">
+<color rgba="0.8 0.8 0.8 1.0"/>
+</material>
+</visual>
+<collision>
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
File: onshape/humanoid_v1/robot.urdf (robot description, URDF)
Before this commit: robot humanoid_v1, 8 links, 7 joints
Links:
- added link lowerlegx, mass 0.516036; collision cylinder length=0.018 radius=0.024; collision cylinder length=0.02 radius=0.045
- added link lowerlegx_2, mass 0.516036; collision cylinder length=0.018 radius=0.024; collision cylinder length=0.02 radius=0.045
- added link lowerlegz, mass 0.602796; collision cylinder length=0.018 radius=0.024; collision cylinder length=0.02 radius=0.045
- added link lowerlegz_2, mass 0.602796; collision cylinder length=0.018 radius=0.024; collision cylinder length=0.02 radius=0.045
- link base: geometry collision box size=0.02 0.02 0.4; collision box size=0.02 0.02 0.4
- link upperlegx: geometry collision cylinder length=0.018 radius=0.024; collision cylinder length=0.02 radius=0.045
- link upperlegx_2: geometry collision cylinder length=0.018 radius=0.024; collision cylinder length=0.02 radius=0.045
- link upperlegy: geometry collision cylinder length=0.018 radius=0.024; collision cylinder length=0.02 radius=0.045
- link upperlegy_2: geometry collision cylinder length=0.018 radius=0.024; collision cylinder length=0.02 radius=0.045
- link upperlegz: geometry collision cylinder length=0.018 radius=0.024; collision cylinder length=0.02 radius=0.045
- link upperlegz_copy_1: geometry collision cylinder length=0.018 radius=0.024; collision cylinder length=0.02 radius=0.045
Joints:
- added joint lowerleg_x_l: type revolute, parent upperlegz_copy_1, child lowerlegx_2, origin xyz=-0.037 -2.52021e-17 0.288 rpy=1.5708 4.44089e-16 1.5708, axis 0 0 1, limit lower=-1.5708 upper=1.5708 effort=1 velocity=20
- added joint lowerleg_x_r: type revolute, parent upperlegz, child lowerlegx, origin xyz=0.037 3.33978e-19 0.288 rpy=1.5708 4.44089e-16 -1.5708, axis 0 0 1, limit lower=-1.5708 upper=1.5708 effort=1 velocity=20
- added joint lowerleg_z_l: type revolute, parent lowerlegx_2, child lowerlegz_2, origin xyz=6.96665e-17 0.14 0.037 rpy=1.5708 -1.5708 0, axis 0 0 1, limit lower=-1.5708 upper=1.5708 effort=1 velocity=20
- added joint lowerleg_z_r: type revolute, parent lowerlegx, child lowerlegz, origin xyz=5.60836e-19 0.14 0.037 rpy=1.5708 1.5708 0, axis 0 0 1, limit lower=-1.5708 upper=1.5708 effort=1 velocity=20
