Commit message: ADD: add lower body model

File: install/humanoid_v1/share/humanoid_v1/urdf/robot.urdf.xacro (robot description, xacro)
@@ -7,4 +7,59 @@
 </joint>
 <link name="base">
+<!-- Shapes for part_2 -->
+<collision>
+<origin xyz="0.04 1.88738e-17 -0.056" rpy="-3.14159 -1.5708 0" />
+<geometry>
+<cylinder length="0.022" radius="0.036" />
+</geometry>
+</collision>
+<!-- Shapes for part_1 -->
+<collision>
+<origin xyz="0.034 0 -0.056" rpy="-3.14159 -1.5708 0" />
+<geometry>
+<cylinder length="0.018" radius="0.024" />
+</geometry>
+</collision>
+<!-- Shapes for extrusion_400mm -->
+<collision>
+<origin xyz="0.065 -0.06 0.21" rpy="0 -0 0" />
+<geometry>
+<box size="0.02 0.02 0.4" />
+</geometry>
+</collision>
+<collision>
+<origin xyz="-0.065 -0.06 0.21" rpy="0 -0 0" />
+<geometry>
+<box size="0.02 0.02 0.4" />
+</geometry>
+</collision>
+<!-- Shapes for motor_shell -->
+<collision>
+<origin xyz="0.035 0 -0.056" rpy="-0 -1.5708 0" />
+<geometry>
+<cylinder length="0.03" radius="0.045" />
+</geometry>
+</collision>
+<!-- Shapes for motor_shell -->
+<collision>
+<origin xyz="-0.035 6.93889e-18 -0.056" rpy="-3.14159 -1.5708 0" />
+<geometry>
+<cylinder length="0.03" radius="0.045" />
+</geometry>
+</collision>
+<!-- Shapes for housing -->
+<collision>
+<origin xyz="-0.066 6.93889e-18 -0.056" rpy="-3.14159 -1.5708 0" />
+<geometry>
+<cylinder length="0.02" radius="0.045" />
+</geometry>
+</collision>
+<!-- Shapes for housing -->
+<collision>
+<origin xyz="0.066 0 -0.056" rpy="-0 -1.5708 0" />
+<geometry>
+<cylinder length="0.02" radius="0.045" />
+</geometry>
+</collision>
 <!-- Shapes for extrusion_150mm -->
 <collision>
@@ -20,239 +75,156 @@
 </geometry>
 </collision>
-<!-- Shapes for housing -->
-<collision>
-<origin xyz="-0.05 6.73073e-18 -0.056" rpy="1.5708 -0 1.5708" />
-<geometry>
-<cylinder length="0.02" radius="0.045" />
+<!-- Shapes for extrusion_100mm -->
+<collision>
+<origin xyz="0.065 0 0" rpy="0 -0 0" />
+<geometry>
+<box size="0.02 0.1 0.02" />
+</geometry>
+</collision>
+<collision>
+<origin xyz="-0.065 0 0" rpy="0 -0 0" />
+<geometry>
+<box size="0.02 0.1 0.02" />
+</geometry>
+</collision>
+<!-- Shapes for housing -->
+<collision>
+<origin xyz="-0.066 6.93889e-18 -0.056" rpy="-3.14159 -1.5708 0" />
+<geometry>
+<cylinder length="0.02" radius="0.045" />
+</geometry>
+</collision>
+<!-- Shapes for extrusion_150mm -->
+<collision>
+<origin xyz="0 0.06 0" rpy="0 -0 0" />
+<geometry>
+<box size="0.15 0.02 0.02" />
+</geometry>
+</collision>
+<collision>
+<origin xyz="0 -0.06 0" rpy="0 -0 0" />
+<geometry>
+<box size="0.15 0.02 0.02" />
 </geometry>
 </collision>
 <!-- Shapes for part_2 -->
 <collision>
-<origin xyz="0.04 1.88738e-17 -0.056" rpy="-3.14159 -1.5708 0" />
+<origin xyz="-0.04 -1.56752e-17 -0.056" rpy="4.17605e-18 -1.5708 0" />
 <geometry>
 <cylinder length="0.022" radius="0.036" />
 </geometry>
 </collision>
+<!-- Shapes for housing -->
+<collision>
+<origin xyz="-0.066 6.93889e-18 -0.056" rpy="-3.14159 -1.5708 0" />
+<geometry>
+<cylinder length="0.02" radius="0.045" />
+</geometry>
+</collision>
+<!-- Shapes for extrusion_400mm -->
+<collision>
+<origin xyz="0.065 -0.06 0.21" rpy="0 -0 0" />
+<geometry>
+<box size="0.02 0.02 0.4" />
+</geometry>
+</collision>
+<collision>
+<origin xyz="-0.065 -0.06 0.21" rpy="0 -0 0" />
+<geometry>
+<box size="0.02 0.02 0.4" />
+</geometry>
+</collision>
+<!-- Shapes for housing -->
+<collision>
+<origin xyz="0.066 0 -0.056" rpy="-0 -1.5708 0" />
+<geometry>
+<cylinder length="0.02" radius="0.045" />
+</geometry>
+</collision>
+<!-- Shapes for extrusion_100mm -->
+<collision>
+<origin xyz="0.065 0 0" rpy="0 -0 0" />
+<geometry>
+<box size="0.02 0.1 0.02" />
+</geometry>
+</collision>
+<collision>
+<origin xyz="-0.065 0 0" rpy="0 -0 0" />
+<geometry>
+<box size="0.02 0.1 0.02" />
+</geometry>
+</collision>
+<!-- Shapes for part_1 -->
+<collision>
+<origin xyz="-0.034 0 -0.056" rpy="-0 -1.5708 0" />
+<geometry>
+<cylinder length="0.018" radius="0.024" />
+</geometry>
+</collision>
+<!-- Shapes for housing -->
+<collision>
+<origin xyz="0.066 0 -0.056" rpy="-0 -1.5708 0" />
+<geometry>
+<cylinder length="0.02" radius="0.045" />
+</geometry>
+</collision>
+<visual>
+<origin xyz="0 0 0" rpy="0 -0 0" />
+<geometry>
+<mesh filename="package://humanoid_v1/meshes/base_visual.stl"/>
+</geometry>
+<material name="base_material">
+<color rgba="0.8 0.8 0.8 1.0"/>
+</material>
+</visual>
+<collision>
+<origin xyz="0 0 0" rpy="0 -0 0" />
+<geometry>
+<mesh filename="package://humanoid_v1/meshes/base_collision.stl"/>
+</geometry>
+<material name="base_material">
+<color rgba="0.5 0.5 0.5 1.0"/>
+</material>
+</collision>
+<inertial>
+<origin xyz="6.62475e-18 -0.010053 -0.00364106" rpy="0 0 0"/>
+<mass value="2.09484" />
+<inertia ixx="0.0277752" ixy="4.21566e-12"  ixz="1.5992e-18" iyy="0.0322146" iyz="0.00449915" izz="0.00921242" />
+</inertial>
+</link>
+<link name="upperlegx">
+<!-- Shapes for part_1 -->
+<collision>
+<origin xyz="0.0315 -4.9426e-15 -0.052" rpy="-1.5708 1.80744e-13 1.5708" />
+<geometry>
+<cylinder length="0.018" radius="0.024" />
+</geometry>
+</collision>
+<!-- Shapes for housing -->
+<collision>
+<origin xyz="-0.0005 -4.8353e-15 -0.052" rpy="1.5708 1.22125e-15 1.5708" />
+<geometry>
+<cylinder length="0.02" radius="0.045" />
+</geometry>
+</collision>
+<!-- Shapes for motor_shell -->
+<collision>
+<origin xyz="0.0305 -5.23454e-15 -0.052" rpy="1.5708 1.22125e-15 1.5708" />
+<geometry>
+<cylinder length="0.03" radius="0.045" />
+</geometry>
+</collision>
+<!-- Shapes for housing -->
+<collision>
+<origin xyz="-0.0005 -4.8353e-15 -0.052" rpy="1.5708 1.22125e-15 1.5708" />
+<geometry>
+<cylinder length="0.02" radius="0.045" />
+</geometry>
+</collision>
 <!-- Shapes for part_2 -->
 <collision>
-<origin xyz="-0.04 -1.56752e-17 -0.056" rpy="4.17605e-18 -1.5708 0" />
+<origin xyz="0.0255 -4.87277e-15 -0.052" rpy="-1.5708 1.57763e-13 1.5708" />
 <geometry>
 <cylinder length="0.022" radius="0.036" />
-</geometry>
-</collision>
-<!-- Shapes for part_1 -->
-<collision>
-<origin xyz="0.034 0 -0.056" rpy="-3.14159 -1.5708 0" />
-<geometry>
-<cylinder length="0.018" radius="0.024" />
-</geometry>
-</collision>
-<!-- Shapes for housing -->
-<collision>
-<origin xyz="-0.066 6.93889e-18 -0.056" rpy="-3.14159 -1.5708 0" />
-<geometry>
-<cylinder length="0.02" radius="0.045" />
-</geometry>
-</collision>
-<!-- Shapes for extrusion_400mm -->
-<collision>
-<origin xyz="0.065 -0.06 0.21" rpy="0 -0 0" />
-<geometry>
-<box size="0.02 0.02 0.4" />
-</geometry>
-</collision>
-<collision>
-<origin xyz="-0.065 -0.06 0.21" rpy="0 -0 0" />
-<geometry>
-<box size="0.02 0.02 0.4" />
-</geometry>
-</collision>
-<!-- Shapes for housing -->
-<collision>
-<origin xyz="0.05 -6.73073e-18 -0.056" rpy="1.5708 -0 -1.5708" />
-<geometry>
-<cylinder length="0.02" radius="0.045" />
-</geometry>
-</collision>
-<!-- Shapes for extrusion_400mm -->
-<collision>
-<origin xyz="0.065 -0.06 0.21" rpy="0 -0 0" />
-<geometry>
-<box size="0.02 0.02 0.4" />
-</geometry>
-</collision>
-<collision>
-<origin xyz="-0.065 -0.06 0.21" rpy="0 -0 0" />
-<geometry>
-<box size="0.02 0.02 0.4" />
-</geometry>
-</collision>
-<!-- Shapes for motor_shell -->
-<collision>
-<origin xyz="0.035 0 -0.056" rpy="-0 -1.5708 0" />
-<geometry>
-<cylinder length="0.03" radius="0.045" />
-</geometry>
-</collision>
-<!-- Shapes for housing -->
-<collision>
-<origin xyz="0.066 0 -0.056" rpy="-0 -1.5708 0" />
-<geometry>
-<cylinder length="0.02" radius="0.045" />
-</geometry>
-</collision>
-<!-- Shapes for motor_shell -->
-<collision>
-<origin xyz="-0.035 6.93889e-18 -0.056" rpy="-3.14159 -1.5708 0" />
-<geometry>
-<cylinder length="0.03" radius="0.045" />
-</geometry>
-</collision>
-<!-- Shapes for extrusion_100mm -->
-<collision>
-<origin xyz="0.065 0 0" rpy="0 -0 0" />
-<geometry>
-<box size="0.02 0.1 0.02" />
-</geometry>
-</collision>
-<collision>
-<origin xyz="-0.065 0 0" rpy="0 -0 0" />
-<geometry>
-<box size="0.02 0.1 0.02" />
-</geometry>
-</collision>
-<!-- Shapes for housing -->
-<collision>
-<origin xyz="-0.066 6.93889e-18 -0.056" rpy="-3.14159 -1.5708 0" />
-<geometry>
-<cylinder length="0.02" radius="0.045" />
-</geometry>
-</collision>
-<!-- Shapes for housing -->
-<collision>
-<origin xyz="0.066 0 -0.056" rpy="-0 -1.5708 0" />
-<geometry>
-<cylinder length="0.02" radius="0.045" />
-</geometry>
-</collision>
-<!-- Shapes for part_1 -->
-<collision>
-<origin xyz="-0.034 0 -0.056" rpy="-0 -1.5708 0" />
-<geometry>
-<cylinder length="0.018" radius="0.024" />
-</geometry>
-</collision>
-<!-- Shapes for housing -->
-<collision>
-<origin xyz="-0.05 6.73073e-18 -0.056" rpy="1.5708 -0 1.5708" />
-<geometry>
-<cylinder length="0.02" radius="0.045" />
-</geometry>
-</collision>
-<!-- Shapes for extrusion_150mm -->
-<collision>
-<origin xyz="0 0.06 0" rpy="0 -0 0" />
-<geometry>
-<box size="0.15 0.02 0.02" />
-</geometry>
-</collision>
-<collision>
-<origin xyz="0 -0.06 0" rpy="0 -0 0" />
-<geometry>
-<box size="0.15 0.02 0.02" />
-</geometry>
-</collision>
-<!-- Shapes for housing -->
-<collision>
-<origin xyz="0.05 -6.73073e-18 -0.056" rpy="1.5708 -0 -1.5708" />
-<geometry>
-<cylinder length="0.02" radius="0.045" />
-</geometry>
-</collision>
-<!-- Shapes for extrusion_100mm -->
-<collision>
-<origin xyz="0.065 0 0" rpy="0 -0 0" />
-<geometry>
-<box size="0.02 0.1 0.02" />
-</geometry>
-</collision>
-<collision>
-<origin xyz="-0.065 0 0" rpy="0 -0 0" />
-<geometry>
-<box size="0.02 0.1 0.02" />
-</geometry>
-</collision>
-<!-- Shapes for housing -->
-<collision>
-<origin xyz="0.066 0 -0.056" rpy="-0 -1.5708 0" />
-<geometry>
-<cylinder length="0.02" radius="0.045" />
-</geometry>
-</collision>
-<!-- Shapes for housing -->
-<collision>
-<origin xyz="-0.066 6.93889e-18 -0.056" rpy="-3.14159 -1.5708 0" />
-<geometry>
-<cylinder length="0.02" radius="0.045" />
-</geometry>
-</collision>
-<visual>
-<origin xyz="0 0 0" rpy="0 -0 0" />
-<geometry>
-<mesh filename="package://humanoid_v1/meshes/base_visual.stl"/>
-</geometry>
-<material name="base_material">
-<color rgba="0.8 0.8 0.8 1.0"/>
-</material>
-</visual>
-<collision>
-<origin xyz="0 0 0" rpy="0 -0 0" />
-<geometry>
-<mesh filename="package://humanoid_v1/meshes/base_collision.stl"/>
-</geometry>
-<material name="base_material">
-<color rgba="0.5 0.5 0.5 1.0"/>
-</material>
-</collision>
-<inertial>
-<origin xyz="7.77955e-18 -0.010053 -0.00364106" rpy="0 0 0"/>
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
File: onshape/humanoid_v1/robot.urdf (robot description, URDF)
Before this commit: robot humanoid_v1, 12 links, 11 joints
Links:
- added link feetx, mass 0.0599595; collision mesh filename=package:///feetx_collision.stl; visual mesh filename=package:///feetx_visual.stl
- added link feetx_copy_1, mass 0.0599594; collision mesh filename=package:///feetx_copy_1_collision.stl; visual mesh filename=package:///feetx_copy_1_visual.stl
- added link feety, mass 1.93667; collision cylinder length=0.02 radius=0.045; collision cylinder length=0.02 radius=0.045
- added link feety_2, mass 1.93667; collision cylinder length=0.02 radius=0.045; collision cylinder length=0.02 radius=0.045
- link base: geometry collision box size=0.02 0.02 0.4; collision box size=0.02 0.02 0.4
- link lowerlegx: mass 0.516036 -> 0.371026; geometry collision cylinder length=0.02 radius=0.045; collision cylinder length=0.02 radius=0.045
- link lowerlegx_2: mass 0.516036 -> 0.371026; geometry collision cylinder length=0.02 radius=0.045; collision cylinder length=0.02 radius=0.045
- link lowerlegz: mass 0.602796 -> 0.457786; geometry collision cylinder length=0.02 radius=0.045; collision cylinder length=0.02 radius=0.045
- link lowerlegz_2: mass 0.602796 -> 0.457786; geometry collision cylinder length=0.02 radius=0.045; collision cylinder length=0.02 radius=0.045
Joints:
- added joint feet_x_l: type revolute, parent lowerlegz_2, child feetx_copy_1, origin xyz=0.0155 -1.48094e-17 -0.2 rpy=-1.5708 -2.95823e-30 1.5708, axis 0 0 1, limit lower=-1.5708 upper=1.5708 effort=1 velocity=20
- added joint feet_x_r: type revolute, parent lowerlegz, child feetx, origin xyz=0.0155 -1.75994e-16 -0.2 rpy=1.5708 -5.24209e-17 -1.5708, axis 0 0 1, limit lower=-1.5708 upper=1.5708 effort=1 velocity=20
- added joint feet_y_l: type revolute, parent feetx_copy_1, child feety_2, origin xyz=0.048 0.0398251 0.0140842 rpy=2.05391e-15 -1.5708 0, axis 0 0 1, limit lower=-1.5708 upper=1.5708 effort=1 velocity=20
- added joint feet_y_r: type revolute, parent feetx, child feety, origin xyz=0.048 -0.0398251 0.0140842 rpy=-3.14159 1.5708 0, axis 0 0 1, limit lower=-1.5708 upper=1.5708 effort=1 velocity=20
- joint lowerleg_z_r: origin xyz=5.60836e-19 0.14 0.037 rpy=1.5708 1.5708 0 -> xyz=-1.3317e-17 0.14 0.037 rpy=1.5708 -1.5708 0
