Commit message: ADD: add correct joint limit

File: install/humanoid_v1/share/humanoid_v1/urdf/robot.urdf.xacro (robot description, xacro)
@@ -55,4 +55,5 @@
 </geometry>
 </collision>
+<!-- Shapes for cycloidal_disk -->
 <!-- Shapes for housing -->
 <collision>
@@ -95,4 +96,5 @@
 </geometry>
 </collision>
+<!-- Shapes for cycloidal_disk -->
 <!-- Shapes for extrusion_150mm -->
 <collision>
@@ -142,4 +144,5 @@
 </geometry>
 </collision>
+<!-- Shapes for cycloidal_disk -->
 <!-- Shapes for extrusion_100mm -->
 <collision>
@@ -155,4 +158,5 @@
 </geometry>
 </collision>
+<!-- Shapes for cycloidal_disk -->
 <!-- Shapes for part_1 -->
 <collision>
@@ -188,7 +192,7 @@
 </collision>
 <inertial>
-<origin xyz="6.62475e-18 -0.010053 -0.00364106" rpy="0 0 0"/>
-<mass value="2.09484" />
-<inertia ixx="0.0277752" ixy="4.21566e-12"  ixz="1.5992e-18" iyy="0.0322146" iyz="0.00449915" izz="0.00921242" />
+<origin xyz="2.1706e-17 -0.0296036 0.154811" rpy="0 0 0"/>
+<mass value="5.09484" />
+<inertia ixx="0.140764" ixy="0.00418147"  ixz="4.66207e-17" iyy="0.230113" iyz="0.0155201" izz="0.0977939" />
 </inertial>
 </link>
@@ -196,26 +200,28 @@
 <!-- Shapes for part_1 -->
 <collision>
-<origin xyz="0.0315 -4.9426e-15 -0.052" rpy="-1.5708 1.80744e-13 1.5708" />
+<origin xyz="0.0315 -6.45678e-15 -0.052" rpy="-1.5708 2.22937e-13 1.5708" />
 <geometry>
 <cylinder length="0.018" radius="0.024" />
 </geometry>
 </collision>
-<!-- Shapes for housing -->
-<collision>
-<origin xyz="-0.0005 -4.8353e-15 -0.052" rpy="1.5708 1.22125e-15 1.5708" />
-<geometry>
-<cylinder length="0.02" radius="0.045" />
-</geometry>
-</collision>
-<!-- Shapes for motor_shell -->
-<collision>
-<origin xyz="0.0305 -5.23454e-15 -0.052" rpy="1.5708 1.22125e-15 1.5708" />
-<geometry>
-<cylinder length="0.03" radius="0.045" />
-</geometry>
-</collision>
-<!-- Shapes for housing -->
-<collision>
-<origin xyz="-0.0005 -4.8353e-15 -0.052" rpy="1.5708 1.22125e-15 1.5708" />
+<!-- Shapes for cycloidal_disk -->
+<!-- Shapes for cycloidal_disk -->
+<!-- Shapes for housing -->
+<collision>
+<origin xyz="-0.0005 -6.25139e-15 -0.052" rpy="1.5708 3.60869e-14 1.5708" />
+<geometry>
+<cylinder length="0.02" radius="0.045" />
+</geometry>
+</collision>
+<!-- Shapes for motor_shell -->
+<collision>
+<origin xyz="0.0305 -7.52653e-15 -0.052" rpy="1.5708 3.60869e-14 1.5708" />
+<geometry>
+<cylinder length="0.03" radius="0.045" />
+</geometry>
+</collision>
+<!-- Shapes for housing -->
+<collision>
+<origin xyz="-0.0005 -6.25139e-15 -0.052" rpy="1.5708 3.60869e-14 1.5708" />
 <geometry>
 <cylinder length="0.02" radius="0.045" />
@@ -224,5 +230,5 @@
 <!-- Shapes for part_2 -->
 <collision>
-<origin xyz="0.0255 -4.87277e-15 -0.052" rpy="-1.5708 1.57763e-13 1.5708" />
+<origin xyz="0.0255 -6.48204e-15 -0.052" rpy="-1.5708 2.00622e-13 1.5708" />
 <geometry>
 <cylinder length="0.022" radius="0.036" />
@@ -231,5 +237,5 @@
 <!-- Shapes for housing -->
 <collision>
-<origin xyz="-0.0005 -4.8353e-15 -0.052" rpy="1.5708 1.22125e-15 1.5708" />
+<origin xyz="-0.0005 -6.25139e-15 -0.052" rpy="1.5708 3.60869e-14 1.5708" />
 <geometry>
 <cylinder length="0.02" radius="0.045" />
@@ -261,7 +267,8 @@
 </link>
 <link name="upperlegy">
+<!-- Shapes for cycloidal_disk -->
 <!-- Shapes for part_2 -->
 <collision>
-<origin xyz="-1.74434e-16 0.099 -0.0175" rpy="-1.5708 -1.68759e-14 7.69755e-15" />
+<origin xyz="-9.63409e-15 0.099 -0.0175" rpy="-1.5708 -1.68759e-14 7.69755e-15" />
 <geometry>
 <cylinder length="0.022" radius="0.036" />
@@ -270,12 +277,12 @@
 <!-- Shapes for housing -->
 <collision>
-<origin xyz="-3.79141e-16 0.125 -0.0175" rpy="1.5708 3.15544e-30 7.69755e-15" />
-<geometry>
-<cylinder length="0.02" radius="0.045" />
-</geometry>
-</collision>
-<!-- Shapes for housing -->
-<collision>
-<origin xyz="-3.79141e-16 0.125 -0.0175" rpy="1.5708 3.15544e-30 7.69755e-15" />
+<origin xyz="-9.84879e-15 0.125 -0.0175" rpy="1.5708 -1.57772e-30 7.69755e-15" />
+<geometry>
+<cylinder length="0.02" radius="0.045" />
+</geometry>
+</collision>
+<!-- Shapes for housing -->
+<collision>
+<origin xyz="-9.84879e-15 0.125 -0.0175" rpy="1.5708 -1.57772e-30 7.69755e-15" />
 <geometry>
 <cylinder length="0.02" radius="0.045" />
@@ -284,5 +291,5 @@
 <!-- Shapes for part_1 -->
 <collision>
-<origin xyz="-1.27787e-16 0.093 -0.0175" rpy="-1.5708 3.15544e-30 7.69755e-15" />
+<origin xyz="-9.58944e-15 0.093 -0.0175" rpy="-1.5708 -1.57772e-30 7.69755e-15" />
 <geometry>
 <cylinder length="0.018" radius="0.024" />
@@ -291,12 +298,13 @@
 <!-- Shapes for motor_shell -->
 <collision>
-<origin xyz="-1.30192e-16 0.094 -0.0175" rpy="1.5708 3.15544e-30 7.69755e-15" />
-<geometry>
-<cylinder length="0.03" radius="0.045" />
-</geometry>
-</collision>
-<!-- Shapes for housing -->
-<collision>
-<origin xyz="-3.79141e-16 0.125 -0.0175" rpy="1.5708 3.15544e-30 7.69755e-15" />
+<origin xyz="-9.61016e-15 0.094 -0.0175" rpy="1.5708 -1.57772e-30 7.69755e-15" />
+<geometry>
+<cylinder length="0.03" radius="0.045" />
+</geometry>
+</collision>
+<!-- Shapes for cycloidal_disk -->
+<!-- Shapes for housing -->
+<collision>
+<origin xyz="-9.84879e-15 0.125 -0.0175" rpy="1.5708 -1.57772e-30 7.69755e-15" />
 <geometry>
 <cylinder length="0.02" radius="0.045" />
@@ -322,5 +330,5 @@
 </collision>
 <inertial>
-<origin xyz="-3.43844e-09 0.109524 -0.0175" rpy="0 0 0"/>
+<origin xyz="-3.43845e-09 0.109524 -0.0175" rpy="0 0 0"/>
 <mass value="0.65579" />
 <inertia ixx="0.000501677" ixy="-1.06691e-07"  ixz="-1.61313e-12" iyy="0.000618053" iyz="2.08745e-12" izz="0.000501763" />
@@ -328,14 +336,23 @@
 </link>
 <link name="upperlegz">
-<!-- Shapes for motor_shell -->
-<collision>
-<origin xyz="-0.011 1.22216e-18 0.288" rpy="-0 -1.5708 0" />
-<geometry>
-<cylinder length="0.03" radius="0.045" />
-</geometry>
-</collision>
+<!-- Shapes for extrusion__length_0.2+meter -->
+<collision>
+<origin xyz="-0.02 2.84367e-20 0.108" rpy="-3.14159 -1.5708 0" />
+<geometry>
+<box size="0.2 0.02 0.02" />
+</geometry>
+</collision>
+<!-- Shapes for motor_shell -->
+<collision>
+<origin xyz="-0.011 -3.82134e-19 0.288" rpy="-0 -1.5708 0" />
+<geometry>
+<cylinder length="0.03" radius="0.045" />
+</geometry>
+</collision>
+<!-- Shapes for cycloidal_disk -->
+<!-- Shapes for cycloidal_disk -->
 <!-- Shapes for part_2 -->
 <collision>
-<origin xyz="-0.006 -1.60178e-18 0.288" rpy="-3.14159 -1.5708 0" />
+<origin xyz="-0.006 -3.20607e-18 0.288" rpy="-3.14159 -1.5708 0" />
 <geometry>
 <cylinder length="0.022" radius="0.036" />
@@ -344,19 +361,26 @@
 <!-- Shapes for housing -->
 <collision>
-<origin xyz="0.02 1.22216e-18 0.288" rpy="-0 -1.5708 0" />
-<geometry>
-<cylinder length="0.02" radius="0.045" />
-</geometry>
-</collision>
-<!-- Shapes for housing -->
-<collision>
-<origin xyz="0.02 1.22216e-18 0.288" rpy="-0 -1.5708 0" />
-<geometry>
-<cylinder length="0.02" radius="0.045" />
-</geometry>
-</collision>
-<!-- Shapes for housing -->
-<collision>
-<origin xyz="0.02 1.22216e-18 0.288" rpy="-0 -1.5708 0" />
+<origin xyz="0.02 -3.82134e-19 0.288" rpy="-0 -1.5708 0" />
+<geometry>
+<cylinder length="0.02" radius="0.045" />
+</geometry>
+</collision>
+<!-- Shapes for extrusion__length_0.2+meter -->
+<collision>
+<origin xyz="0.02 -5.44764e-19 0.108" rpy="-3.14159 -1.5708 0" />
+<geometry>
+<box size="0.2 0.02 0.02" />
+</geometry>
+</collision>
+<!-- Shapes for housing -->
+<collision>
+<origin xyz="0.02 -3.82134e-19 0.288" rpy="-0 -1.5708 0" />
+<geometry>
+<cylinder length="0.02" radius="0.045" />
+</geometry>
+</collision>
+<!-- Shapes for housing -->
+<collision>
+<origin xyz="0.02 -3.82134e-19 0.288" rpy="-0 -1.5708 0" />
 <geometry>
 <cylinder length="0.02" radius="0.045" />
@@ -365,5 +389,5 @@
 <!-- Shapes for part_1 -->
 <collision>
-<origin xyz="-0.012 1.22134e-17 0.288" rpy="-3.14159 -1.5708 0" />
+<origin xyz="-0.012 1.06091e-17 0.288" rpy="-3.14159 -1.5708 0" />
 <geometry>
 <cylinder length="0.018" radius="0.024" />
@@ -395,32 +419,34 @@
 </link>
 <link name="lowerlegx">
-<!-- Shapes for housing -->
-<collision>
-<origin xyz="1.19838e-19 0.123 0.037" rpy="1.5708 1.5708 0" />
-<geometry>
-<cylinder length="0.02" radius="0.045" />
-</geometry>
-</collision>
-<!-- Shapes for housing -->
-<collision>
-<origin xyz="1.19838e-19 0.123 0.037" rpy="1.5708 1.5708 0" />
-<geometry>
-<cylinder length="0.02" radius="0.045" />
-</geometry>
-</collision>
-<!-- Shapes for housing -->
-<collision>
-<origin xyz="1.19838e-19 0.123 0.037" rpy="1.5708 1.5708 0" />
-<geometry>
-<cylinder length="0.02" radius="0.045" />
-</geometry>
-</collision>
-<!-- Shapes for motor_shell -->
-<collision>
-<origin xyz="1.19838e-19 0.092 0.037" rpy="1.5708 1.5708 0" />
-<geometry>
-<cylinder length="0.03" radius="0.045" />
-</geometry>
-</collision>
+<!-- Shapes for cycloidal_disk -->
+<!-- Shapes for housing -->
+<collision>
+<origin xyz="-3.10811e-30 0.123 0.037" rpy="1.5708 1.5708 0" />
+<geometry>
+<cylinder length="0.02" radius="0.045" />
+</geometry>
+</collision>
+<!-- Shapes for housing -->
+<collision>
+<origin xyz="-3.10811e-30 0.123 0.037" rpy="1.5708 1.5708 0" />
+<geometry>
+<cylinder length="0.02" radius="0.045" />
+</geometry>
+</collision>
+<!-- Shapes for housing -->
+<collision>
+<origin xyz="-3.10811e-30 0.123 0.037" rpy="1.5708 1.5708 0" />
+<geometry>
+<cylinder length="0.02" radius="0.045" />
+</geometry>
+</collision>
+<!-- Shapes for motor_shell -->
+<collision>
+<origin xyz="-3.01029e-30 0.092 0.037" rpy="1.5708 1.5708 0" />
+<geometry>
+<cylinder length="0.03" radius="0.045" />
+</geometry>
+</collision>
+<!-- Shapes for cycloidal_disk -->
 <visual>
 <origin xyz="0 0 0" rpy="0 -0 0" />
@@ -450,26 +476,35 @@
 <!-- Shapes for housing -->
 <collision>
-<origin xyz="-0.0015 -3.79149e-16 -0.2" rpy="3.14159 1.5708 0" />
-<geometry>
-<cylinder length="0.02" radius="0.045" />
-</geometry>
-</collision>
-<!-- Shapes for housing -->
-<collision>
-<origin xyz="-0.0015 -3.79149e-16 -0.2" rpy="3.14159 1.5708 0" />
-<geometry>
-<cylinder length="0.02" radius="0.045" />
-</geometry>
-</collision>
-<!-- Shapes for housing -->
-<collision>
-<origin xyz="-0.0015 -3.79149e-16 -0.2" rpy="3.14159 1.5708 0" />
-<geometry>
-<cylinder length="0.02" radius="0.045" />
-</geometry>
-</collision>
-<!-- Shapes for motor_shell -->
-<collision>
-<origin xyz="-0.0325 -3.79149e-16 -0.2" rpy="3.14159 1.5708 0" />
+<origin xyz="-0.0015 -2.36789e-18 -0.2" rpy="3.14159 1.5708 0" />
+<geometry>
+<cylinder length="0.02" radius="0.045" />
+</geometry>
+</collision>
+<!-- Shapes for housing -->
+<collision>
+<origin xyz="-0.0015 -2.36789e-18 -0.2" rpy="3.14159 1.5708 0" />
+<geometry>
+<cylinder length="0.02" radius="0.045" />
+</geometry>
+</collision>
+<!-- Shapes for cycloidal_disk -->
+<!-- Shapes for extrusion__length_0.15+meter -->
+<collision>
+<origin xyz="2.77556e-17 1.6263e-19 -0.085" rpy="-0 1.5708 0" />
+<geometry>
+<box size="0.15 0.02 0.02" />
+</geometry>
+</collision>
+<!-- Shapes for housing -->
+<collision>
+<origin xyz="-0.0015 -2.36789e-18 -0.2" rpy="3.14159 1.5708 0" />
+<geometry>
+<cylinder length="0.02" radius="0.045" />
+</geometry>
+</collision>
+<!-- Shapes for cycloidal_disk -->
+<!-- Shapes for motor_shell -->
+<collision>
+<origin xyz="-0.0325 -2.36789e-18 -0.2" rpy="3.14159 1.5708 0" />
 <geometry>
 <cylinder length="0.03" radius="0.045" />
@@ -495,5 +530,5 @@
 </collision>
 <inertial>
-<origin xyz="-0.0111152 -7.92875e-12 -0.158926" rpy="0 0 0"/>
+<origin xyz="-0.0111152 -7.92857e-12 -0.158926" rpy="0 0 0"/>
 <mass value="0.457786" />
 <inertia ixx="0.00222732" ixy="-2.17139e-12"  ixz="-0.000217459" iyy="0.00224323" iyz="5.16092e-09" izz="0.000243554" />
@@ -501,4 +536,11 @@
 </link>
 <link name="feetx">
+<!-- Shapes for feet -->
+<collision>
+<origin xyz="0 0 0" rpy="-1.5708 -1.5708 0" />
+<geometry>
+<sphere radius="0.01" />
+</geometry>
+</collision>
 <visual>
 <origin xyz="0 0 0" rpy="0 -0 0" />
@@ -510,13 +552,4 @@
 </material>
 </visual>
-<collision>
-<origin xyz="0 0 0" rpy="0 -0 0" />
-<geometry>
-<mesh filename="package://humanoid_v1/meshes/feetx_collision.stl"/>
-</geometry>
-<material name="feetx_material">
-<color rgba="0.5 0.5 0.5 1.0"/>
-</material>
-</collision>
 <inertial>
 <origin xyz="0.0223276 -0.0258701 0.00228741" rpy="0 0 0"/>
@@ -533,4 +566,5 @@
 </geometry>
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
File: onshape/humanoid_v1/robot.urdf (robot description, URDF)
Before this commit: robot humanoid_v1, 16 links, 15 joints
Links:
- link base: mass 2.09484 -> 5.09484
- link feetx: geometry collision sphere radius=0.01; visual mesh filename=package:///feetx_visual.stl
- link lowerlegz: geometry collision box size=0.15 0.02 0.02; collision cylinder length=0.02 radius=0.045
- link lowerlegz_2: geometry collision box size=0.15 0.02 0.02; collision cylinder length=0.02 radius=0.045
- link upperlegz: geometry collision box size=0.2 0.02 0.02; collision box size=0.2 0.02 0.02
- link upperlegz_copy_1: geometry collision box size=0.2 0.02 0.02; collision box size=0.2 0.02 0.02
Joints:
- joint feet_x_l: limit lower=-1.5708 upper=1.5708 effort=1 velocity=20 -> lower=-0.785398 upper=0.785398 effort=1 velocity=20
- joint feet_x_r: limit lower=-1.5708 upper=1.5708 effort=1 velocity=20 -> lower=-0.785398 upper=0.785398 effort=1 velocity=20; origin xyz=0.0155 -1.75994e-16 -0.2 rpy=1.5708 -5.24209e-17 -1.5708 -> xyz=0.0155 -2.36789e-18 -0.2 rpy=1.5708 -5.24209e-17 -1.5708
- joint feet_y_l: limit lower=-1.5708 upper=1.5708 effort=1 velocity=20 -> lower=-0.261799 upper=0.261799 effort=1 velocity=20
- joint feet_y_r: limit lower=-1.5708 upper=1.5708 effort=1 velocity=20 -> lower=-0.261799 upper=0.261799 effort=1 velocity=20
- joint lowerleg_x_l: limit lower=-1.5708 upper=1.5708 effort=1 velocity=20 -> lower=-1.74533 upper=0.174533 effort=1 velocity=20
- joint lowerleg_x_r: limit lower=-1.5708 upper=1.5708 effort=1 velocity=20 -> lower=-0.174533 upper=1.74533 effort=1 velocity=20; origin xyz=0.037 3.33978e-19 0.288 rpy=1.5708 4.44089e-16 -1.5708 -> xyz=0.037 9.07461e-19 0.288 rpy=1.5708 9.49411e-16 -1.5708
- joint lowerleg_z_l: limit lower=-1.5708 upper=1.5708 effort=1 velocity=20 -> lower=-0.785398 upper=0.785398 effort=1 velocity=20
- joint lowerleg_z_r: limit lower=-1.5708 upper=1.5708 effort=1 velocity=20 -> lower=-0.785398 upper=0.785398 effort=1 velocity=20; origin xyz=-1.3317e-17 0.14 0.037 rpy=1.5708 -1.5708 0 -> xyz=-3.15544e-30 0.14 0.037 rpy=1.5708 -1.5708 0
- joint upperleg_x_l: limit lower=-6.28319 upper=6.28319 effort=1 velocity=20 -> lower=-1.5708 upper=1.5708 effort=1 velocity=20
- joint upperleg_x_r: limit lower=-6.28319 upper=6.28319 effort=1 velocity=20 -> lower=-1.5708 upper=1.5708 effort=1 velocity=20; origin xyz=0.083 2.90452e-17 -0.056 rpy=1.5708 -3.55271e-15 -1.5708 -> xyz=0.083 2.90452e-17 -0.056 rpy=1.5708 -1.06581e-14 -1.5708
- joint upperleg_y_l: limit lower=-6.28319 upper=6.28319 effort=1 velocity=20 -> lower=-0.261799 upper=1.0472 effort=1 velocity=20; origin xyz=-0.0175 -4.16334e-17 -0.052 rpy=6.12323e-17 -1.5708 0 -> xyz=-0.0175 1.38778e-17 -0.052 rpy=6.12323e-17 -1.5708 0
- joint upperleg_y_r: limit lower=-6.28319 upper=6.28319 effort=1 velocity=20 -> lower=-1.0472 upper=0.261799 effort=1 velocity=20; origin xyz=-0.0175 -4.54498e-15 -0.052 rpy=-3.14159 1.5708 0 -> xyz=-0.0175 -5.52336e-15 -0.052 rpy=-3.14159 1.5708 0
- joint upperleg_z_l: limit lower=-1.5708 upper=1.5708 effort=1 velocity=20 -> lower=-0.785398 upper=0.785398 effort=1 velocity=20; origin xyz=-4.71845e-16 0.142 -0.0175 rpy=-1.5708 -2.15921e-15 7.69755e-15 -> xyz=-2.47025e-15 0.142 -0.0175 rpy=-1.5708 -2.15921e-15 7.69755e-15
- joint upperleg_z_r: limit lower=-1.5708 upper=1.5708 effort=1 velocity=20 -> lower=-0.785398 upper=0.785398 effort=1 velocity=20; origin xyz=-5.27356e-16 0.142 -0.0175 rpy=-1.5708 -1.65983e-14 7.69755e-15 -> xyz=-9.99201e-15 0.142 -0.0175 rpy=-1.5708 1.15338e-14 7.69755e-15
